File: Hardware/Vegan-Greg/GPIO.kicad_sch (KiCad schematic)
At the start: 0 parts

Commit message: vegangreg schem
Parts:
- added D5: RCLAMP3346PQTNT, iclr:RCLAMP3346PQTNT, symbol iclr:RCLAMP3346PQTNT
- added J5: GPIO Breakout, Connector_PinSocket_2.54mm:PinSocket_2x04_P2.54mm_Vertical, symbol Connector:Conn_01x08_Female
- added R40, R41, R42, R43, R44, R45: 10k, Resistor_SMD:R_0402_1005Metric, symbol Device:R_Small
Connections:
- new net +3V3: J5.5 (Pin_5), R40.1, R41.1, R42.1, R43.1, R44.1, R45.1
- new net GND: D5.2 (GND), J5.1 (Pin_1)
- new net GPIO10: D5.4 (K/A_3), J5.2 (Pin_2), R43.2
- new net GPIO5: D5.1 (K/A_1), J5.7 (Pin_7), R44.2
- new net GPIO6: D5.5 (K/A_4), J5.8 (Pin_8), R45.2
- new net GPIO7: D5.6 (K/A_5), J5.6 (Pin_6), R42.2
- new net GPIO8: D5.3 (K/A_2), J5.3 (Pin_3), R41.2
- new net GPIO9: D5.7 (K/A_6), J5.4 (Pin_4), R40.2
