File: Hardware/Vegan-Greg/VeganGreg.kicad_sch (KiCad schematic)
At the start: 39 parts, among them J1 RBUS, U1 ESP32-S3, Y1 R940000171

Commit message: vegangreg schem
Parts:
- added C55: 0.1uF, Capacitor_SMD:C_0402_1005Metric, symbol Device:C_Small
- added R36: 18k, Resistor_SMD:R_0402_1005Metric, symbol Device:R_Small
- added R37: 1.5k, Resistor_SMD:R_0402_1005Metric, symbol Device:R_Small
- added R38: 470, Resistor_SMD:R_0402_1005Metric, symbol Device:R_Small
- added R39: 1k, Resistor_SMD:R_0402_1005Metric, symbol Device:R_Small
- added SERVOLED1: AMBER_LED, LED_SMD:LED_0402_1005Metric, symbol Device:LED_Small
Connections:
- net CAN_RX: now also U1.39 (GPIO34)
- net CAN_TX: now also U1.38 (GPIO33)
- net GND: now also R36.1, R38.1, SERVOLED1.1 (K)
- net GPIO5: now reaches U1.10 (GPIO5/ADC1_CH4)
- net GPIO6: now reaches U1.11 (GPIO6/ADC1_CH5)
- net GPIO7: now reaches U1.12 (GPIO7/ADC1_CH6)
- net GPIO8: now reaches U1.13 (GPIO8/ADC1_CH7)
- net GPIO9: now reaches U1.14 (GPIO9/ADC1_CH8)
- net GPIO10: now reaches U1.15 (GPIO10/ADC1_CH9)
- net BuckPGOOD: now reaches U1.37 (SPICLK_P/GPIO47)
- net BuckPGOOD: now also R36.2
- net Servo0PWM: now reaches U1.41 (GPIO36)
- net BUCK_EN: now reaches U1.43 (GPIO38)
- net +12V renamed 25.2V
- net +16.8V renamed +25.2V
- new net: R39.2, SERVOLED1.2 (A)
- new net +6V: C55.1, R37.2, R39.1
- new net ServoV_LOG: C55.2, R37.1, R38.2
Other:
- added sheet GPIO (GPIO.kicad_sch)
- added sheet gregPart (gregPart.kicad_sch)
- sheet Servo Connectors ports: added Servo_0_PWM; removed none
- sheet buckC ports: added BUCK_EN, PGOOD; removed none
