File: Hardware/Vegan-Greg/buckC.kicad_sch (KiCad schematic)
At the start: 0 parts

Commit message: vegangreg schem
Parts:
- added C12: 1uF, Capacitor_SMD:C_0402_1005Metric, symbol Device:C_Small
- added C18: 4.7uF, Capacitor_SMD:C_0402_1005Metric, symbol Device:C_Small
- added C19, C37: 100uF, Capacitor_Tantalum_SMD:CP_EIA-7360-38_Kemet-E, symbol Device:C_Polarized_Small
- added C28, C29, C31, C32, C33, C36, C38, C39, C40, C41: 47uF, Capacitor_SMD:C_1206_3216Metric, symbol Device:C_Small
- added C30: 100nF, Capacitor_SMD:C_0402_1005Metric, symbol Device:C_Small
- added C34: 0.1uF, Capacitor_SMD:C_0402_1005Metric, symbol Device:C_Small
- added C35: 160pF, Capacitor_SMD:C_0603_1608Metric, symbol Device:C_Small
- added L4: 3.3uH, iclr:IND_SPM10065VT-3R3M-D, symbol Device:L
- added Q1: SSM3K15AMFV,L3F, iclr:SOT-723, symbol Device:Q_NMOS_GSD
- added R20, R22, R28: 10k, Resistor_SMD:R_0402_1005Metric, symbol Device:R_Small
- added R21: 113k, Resistor_SMD:R_0402_1005Metric, symbol Device:R_Small
- added R23: 2.2, Resistor_SMD:R_0402_1005Metric, symbol Device:R_Small
- added R24: 1k, Resistor_SMD:R_0402_1005Metric, symbol Device:R_Small
- added R25: 442k, Resistor_SMD:R_0402_1005Metric, symbol Device:R_Small
- added R26: 200k, Resistor_SMD:R_0402_1005Metric, symbol Device:R_Small
- added R27: 100k, Resistor_SMD:R_0402_1005Metric, symbol Device:R_Small
- added R29: 5.1R, Resistor_SMD:R_0603_1608Metric, symbol Device:R_Small
- added U6: SIC438AED-T1, iclr:SiC437BEDT1GE3, symbol iclr:SiC437BED-T1-GE3
Connections:
- new net: C35.2, R29.1
- new net: C18.2, U6.12 (V_DRV)
- new net: R26.1, U6.20 (MODE_2)
- new net: R27.1, U6.21 (_MODE_1)
- new net: C34.2, R23.2
- new net +16.8V: C19.1, C30.1, C37.1, R28.2, U6.1 (V_IN_1), U6.2 (V_IN_2), U6.22 (VIN_1), U6.26 (VIN_2)
- new net +6V: C28.1, C29.1, C31.1, C32.1, C33.1, C36.2, C38.1, C39.1, C40.1, C41.1, L4.1, R21.2, R25.2, U6.18 (V_OUT)
- new net BOOT: C34.1, U6.23 (BOOT)
- new net BUCK_EN: Q1.1 (G), R24.2
- new net EN: Q1.3 (D), R28.1, U6.19 (EN)
- new net FB: R21.1, R22.2, R25.1, U6.17 (FB)
- new net GND: C12.1, C18.1, C19.2, C28.2, C29.2, C30.2, C31.2, C32.2, C33.2, C36.1, C37.2, C38.2, C39.2, C40.2, C41.2, Q1.2 (S), R22.1, R24.1, R27.2, R29.2, U6.13 (P_GND_3), U6.16 (A_GND), U6.25 (AGND), U6.27 (PGND), U6.29 (P_GND_4), U6.3 (P_GND_1), U6.4 (P_GND_2)
- new net PGOOD: R20.2, U6.14 (P_GOOD)
- new net PHASE: R23.1, U6.24 (PHASE)
- new net SW: C35.1, L4.2, U6.30 (SW_6), U6.5 (SW_1), U6.6 (SW_2), U6.7 (SW_3), U6.8 (SW_4), U6.9 (SW_5)
- new net VDD: C12.2, R20.1, R26.2, U6.15 (VDD)
- no-connect marks 0 -> 3
Other:
- note added: "Backup capacitors, only place if the capacitance is too low"
- note added: "Input Capacitors"
- note added: "Output Capacitors"
- note added: "RC Snubber"
- note added: "SPM10065VT-3R3M-D"
