File: Hardware/Vegan-Greg/gregPart.kicad_sch (KiCad schematic)
At the start: 26 parts, among them J1 Conn_01x06_Socket, U1 TPS61089, U2 LT1762

Commit message: vegangreg schem
Parts:
- removed C1, C10, C11, C7: 22µF, symbol Device:C_Small
- removed C2: 0.1µF, symbol Device:C_Small
- removed C22, C33: 10uF, Capacitor_SMD:C_0402_1005Metric, symbol Device:C_Small
- removed C23, C34: 100nF, Capacitor_SMD:C_0402_1005Metric, symbol Device:C_Small
- removed C3: 2.2µF, symbol Device:C_Small
- removed C4: 1µF, symbol Device:C_Small
- removed C5: 180pF, symbol Device:C_Small
- removed C6: 4.7nF, symbol Device:C_Small
- removed C8: 0.01µF, symbol Device:C_Small
- removed C9: 10µF, symbol Device:C_Small
- removed J1: Conn_01x06_Socket, symbol Connector:Conn_01x06_Socket
- removed JP1: SolderJumper_3_Open, Jumper:SolderJumper-3_P1.3mm_Open_RoundedPad1.0x1.5mm_NumberLabels, symbol Jumper:SolderJumper_3_Open
- removed L1: 1.8µH, symbol Device:L
- removed R1: 301k, symbol Device:R
- removed R2: 127k, symbol Device:R
- removed R3: 17.4k, symbol Device:R
- removed R4: 100k, symbol Device:R
- removed R5: 18k, symbol Device:R
- removed R6: 51k, symbol Device:R
- removed U1: TPS61089, Package_DFN_QFN:Texas_VQFN-RNR0011A-11, symbol Regulator_Switching:TPS61089
- removed U2: LT1762, Package_SO:MSOP-8_3x3mm_P0.65mm, symbol Regulator_Linear:LT1762
- added C42, C49, C50, C51: 22µF, symbol Device:C_Small
- added C43: 1µF, symbol Device:C_Small
- added C44: 0.1µF, symbol Device:C_Small
- added C45: 10uF, Capacitor_SMD:C_0402_1005Metric, symbol Device:C_Small
- added C46: 100nF, Capacitor_SMD:C_0402_1005Metric, symbol Device:C_Small
- added C47: 2.2µF, symbol Device:C_Small
- added C48: 0.01µF, symbol Device:C_Small
- added C52: 180pF, symbol Device:C_Small
- added C53: 10µF, symbol Device:C_Small
- added C54: 4.7nF, symbol Device:C_Small
- added J4: Conn_01x06_Socket, symbol Connector:Conn_01x06_Socket
- added JP2: SolderJumper_3_Open, Jumper:SolderJumper-3_P1.3mm_Open_RoundedPad1.0x1.5mm_NumberLabels, symbol Jumper:SolderJumper_3_Open
- added L5: 1.8µH, symbol Device:L
- added R30: 301k, symbol Device:R
- added R31: 127k, symbol Device:R
- added R32: 17.4k, symbol Device:R
- added R33: 100k, symbol Device:R
- added R34: 51k, symbol Device:R
- added R35: 18k, symbol Device:R
- added U7: LT1762, Package_SO:MSOP-8_3x3mm_P0.65mm, symbol Regulator_Linear:LT1762
- added U8: TPS61089, Package_DFN_QFN:Texas_VQFN-RNR0011A-11, symbol Regulator_Switching:TPS61089
Connections:
- net +12V: now also J4.4 (Pin_4)
- net +3.3V: now also C42.1, L5.1, U8.7 (EN), U8.9 (VIN)
- net GND: now also C42.2, C43.2, C45.2, C46.2, C47.2, C49.2, C50.2, C51.2, C52.2, C53.2, C54.2, J4.1 (Pin_1), J4.2 (Pin_2), R31.2, R33.2, R35.2, U7.4 (GND), U8.5 (GND)
- net LDO5.5V_IN: now also C45.1, C46.1
- net RBUS_uC_V: now also J4.3 (Pin_3)
- net VOut - 5 or 12V: now also C49.1, C50.1, C51.1, R34.1, U8.6 (VOUT)
- new net: C47.1, U8.2 (VCC)
- new net: C44.1, L5.2, R30.1, U8.11 (SW)
- new net: C44.2, U8.10 (BOOT)
- new net: C48.1, C53.1, U7.1 (OUT), U7.2 (ADJ)
- new net: C48.2, U7.3 (BYP)
- new net: C43.1, U7.5 (~{SHDN}), U7.8 (IN)
- new net: C52.1, R32.1, U8.4 (COMP)
- new net: C54.1, R32.2
- new net: JP2.2 (C), R34.2, U8.3 (FB)
- new net: R30.2, U8.1 (FSW)
- new net: JP2.1 (A), R35.1
- new net: R31.1, U8.8 (ILIM)
- new net: JP2.3 (B), R33.1
