File: Hardware/Vegan-Greg/VeganGreg.kicad_pcb (KiCad board)
At the start: 4 copper layers, 16 parts, among them U3 LM66200DRLR, U4 MAX77827AEFD+T, U5 SC4215ASTRT

Commit message: Review Ready
Parts:
- added 12VLED1: RED_LED, Resistor_SMD:R_0402_1005Metric, F.Cu at (24.0, 0.49)
- added 3V3LED1: BLUE_LED, Resistor_SMD:R_0402_1005Metric, F.Cu at (24.0, 2.48)
- added BOOTJUMPER1: Conn_01x02_Male, Connector_PinHeader_2.54mm:PinHeader_1x02_P2.54mm_Vertical, F.Cu at (18.8, 25.1)
- added C1: 10uF, Capacitor_SMD:C_0402_1005Metric, F.Cu at (23.9, 12.4)
- added C10: 0.1uF, Capacitor_SMD:C_0402_1005Metric, F.Cu at (26.8, 20.3)
- added C11: 0.1uF, Capacitor_SMD:C_0402_1005Metric, F.Cu at (29.7, 12.4)
- added C13: 11pF, Capacitor_SMD:C_0402_1005Metric, F.Cu at (29.7, 14.4)
- added C14: 11pF, Capacitor_SMD:C_0402_1005Metric, F.Cu at (29.7, 16.4)
- added C15: 100nF, Capacitor_SMD:C_0402_1005Metric, F.Cu at (4.95, 41.6)
- added C16: 10uF, Capacitor_SMD:C_0402_1005Metric, F.Cu at (4.95, 43.6)
- added C17: 47nF, Capacitor_SMD:C_0402_1005Metric, F.Cu at (4.95, 45.6)
- added C2: 1uF, Capacitor_SMD:C_0402_1005Metric, F.Cu at (23.9, 14.4)
- added C3: 0.1uF, Capacitor_SMD:C_0402_1005Metric, F.Cu at (23.9, 16.4)
- added C4: 1uF, Capacitor_SMD:C_0402_1005Metric, F.Cu at (23.9, 18.3)
- added C5: 0.1uF, Capacitor_SMD:C_0402_1005Metric, F.Cu at (23.9, 20.3)
- added C6: 0.1uF, Capacitor_SMD:C_0402_1005Metric, F.Cu at (26.8, 12.4)
- added C7: 1uF, Capacitor_SMD:C_0402_1005Metric, F.Cu at (26.8, 14.4)
- added C8: 0.1uF, Capacitor_SMD:C_0402_1005Metric, F.Cu at (26.8, 16.4)
- added C9: 10nF, Capacitor_SMD:C_0402_1005Metric, F.Cu at (26.8, 18.3)
- added CRXLED1: ORANGE_LED, Resistor_SMD:R_0402_1005Metric, F.Cu at (24.0, 4.47)
- added CTXLED1: GREEN_LED, Resistor_SMD:R_0402_1005Metric, F.Cu at (24.0, 6.46)
- added D1: SM712_SOT23, Package_TO_SOT_SMD:SOT-23, F.Cu at (8.82, 43.0)
- added D2: SP0503BAHT, Package_TO_SOT_SMD:SOT-143, F.Cu at (35.4, 11.9)
- added ENJUMPER1: Conn_01x02_Male, Connector_PinHeader_2.54mm:PinHeader_1x02_P2.54mm_Vertical, F.Cu at (23.4, 25.1)
- added G***: LOGO, LOGO, F.Cu at (162.9, 89.6)
- added G***: LOGO, iclr:rae_logo_4mm, F.Cu at (185.9, 89.6)
- added H1: MountingHole_Pad, MountingHole:MountingHole_3.2mm_M3_DIN965_Pad, F.Cu at (3.08, 3.08)
- added H2: MountingHole_Pad, MountingHole:MountingHole_3.2mm_M3_DIN965_Pad, F.Cu at (3.08, 10.2)
- added H3: MountingHole_Pad, MountingHole:MountingHole_3.2mm_M3_DIN965_Pad, F.Cu at (3.08, 17.4)
- added H4: MountingHole_Pad, MountingHole:MountingHole_3.2mm_M3_DIN965_Pad, F.Cu at (3.08, 24.5)
- added J1: RBUS, Connector_Molex:Molex_Mini-Fit_Jr_5569-06A2_2x03_P4.20mm_Horizontal, F.Cu at (10.4, 14.4)
- added J2: USB_C_Receptacle_USB2.0, Connector_USB:USB_C_Receptacle_Palconn_UTC16-G, F.Cu at (39.0, 3.62)
- added JP1: TermJP, Jumper:SolderJumper-2_P1.3mm_Open_RoundedPad1.0x1.5mm, F.Cu at (10.1, 35.8)
- added L1: 2.0nH, Inductor_SMD:L_0402_1005Metric, F.Cu at (24.0, 8.46)
- added L2: 20nH, Inductor_SMD:L_0402_1005Metric, F.Cu at (24.0, 10.4)
- added R1: 10K, Resistor_SMD:R_0402_1005Metric, F.Cu at (26.9, 0.49)
- added R10: 60, Resistor_SMD:R_0603_1608Metric, F.Cu at (1.50, 46.9)
- added R11: 5.1k, Resistor_SMD:R_0402_1005Metric, F.Cu at (42.0, 10.5)
- added R12: 5.1k, Resistor_SMD:R_0402_1005Metric, F.Cu at (42.0, 12.5)
- added R13: 5.1k, Resistor_SMD:R_0402_1005Metric, F.Cu at (42.0, 14.5)
- added R18: 1k, Resistor_SMD:R_0402_1005Metric, F.Cu at (29.8, 2.48)
- added R2: 470, Resistor_SMD:R_0402_1005Metric, F.Cu at (26.9, 2.48)
- added R3: 10K, Resistor_SMD:R_0402_1005Metric, F.Cu at (26.9, 4.47)
- added R4: 470, Resistor_SMD:R_0402_1005Metric, F.Cu at (26.9, 6.46)
- added R5: 1k, Resistor_SMD:R_0402_1005Metric, F.Cu at (26.9, 8.46)
- added R6: 499R, Resistor_SMD:R_0402_1005Metric, F.Cu at (26.9, 10.4)
- added R7: 3k, Resistor_SMD:R_0402_1005Metric, F.Cu at (29.8, 0.49)
- added R8: 0, Resistor_SMD:R_0603_1608Metric, F.Cu at (1.50, 41.9)
- added R9: 60, Resistor_SMD:R_0603_1608Metric, F.Cu at (1.50, 44.4)
- added REF**: MountingHole_2.2mm_M2_DIN965_Pad, MountingHole:MountingHole_2.2mm_M2_DIN965_Pad, F.Cu at (188.4, 98.1)
- added REF**: MountingHole_2.2mm_M2_DIN965_Pad, MountingHole:MountingHole_2.2mm_M2_DIN965_Pad, F.Cu at (160.9, 83.1)
- added REF**: MountingHole_2.2mm_M2_DIN965_Pad, MountingHole:MountingHole_2.2mm_M2_DIN965_Pad, F.Cu at (160.9, 98.1)
- added REF**: MountingHole_2.2mm_M2_DIN965_Pad, MountingHole:MountingHole_2.2mm_M2_DIN965_Pad, F.Cu at (188.4, 83.1)
- added TP1: TestPoint, TestPoint:TestPoint_Pad_D1.0mm, F.Cu at (39.0, 11.0)
- added TP10: TestPoint, TestPoint:TestPoint_Pad_D1.0mm, F.Cu at (27.3, 27.4)
- added TP2: TestPoint, TestPoint:TestPoint_Pad_D1.0mm, F.Cu at (39.0, 14.1)
- added TP4: TestPoint, TestPoint:TestPoint_Pad_D1.5mm, F.Cu at (16.1, 35.8)
- added TP5: TestPoint, TestPoint:TestPoint_Pad_D1.5mm, F.Cu at (16.1, 39.4)
- added TP6: TestPoint, TestPoint:TestPoint_Pad_D1.5mm, F.Cu at (16.1, 42.9)
- added TP8: TestPoint, TestPoint:TestPoint_Pad_D1.5mm, F.Cu at (16.1, 46.5)
- added TP9: TestPoint, TestPoint:TestPoint_Pad_D1.0mm, F.Cu at (27.3, 24.3)
- added TXLED1: GREEN_LED, Resistor_SMD:R_0402_1005Metric, F.Cu at (29.8, 4.47)
- added U1: ESP32-S3, iclr:QFN40P700X700X90-57N, F.Cu at (11.8, 27.4)
- added U2: SN65HVD230, Package_SO:SOIC-8_3.9x4.9mm_P1.27mm, F.Cu at (3.73, 37.4)
- added USBLED1: WHITE_LED, Resistor_SMD:R_0402_1005Metric, F.Cu at (42.0, 16.4)
- added Y1: R940000171, Crystal:Crystal_SMD_2016-4Pin_2.0x1.6mm, F.Cu at (1.43, 29.9)
- moved C23 0.33 mm to (175.2, 88.1)
- moved C26 0.33 mm to (176.8, 91.7)
- moved C27 0.33 mm to (176.8, 92.6)
- moved R14 0.33 mm to (168.5, 89.1)
- moved R16 0.33 mm to (178.6, 91.7)
- moved U3 0.33 mm to (167.7, 87.0)
- moved U5 0.33 mm to (178.7, 87.5)
- moved C20 0.33 mm to (169.4, 85.5)
- moved L3 0.33 mm to (172.6, 90.7)
- moved R15 0.33 mm to (172.4, 84.7)
- moved C24 0.33 mm to (179.8, 83.4)
- moved C25 0.33 mm to (177.7, 83.4)
- moved R17 0.33 mm to (180.5, 91.7)
- moved U4 0.33 mm to (172.6, 87.0)
- moved C21 0.33 mm to (170.1, 88.3)
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Routing:
- added copper zone on B.Cu, net GND
- added copper zone on In1.Cu, net GND
Other:
- board outline added: 32.5 x 20 mm
- board text added: "Vegan-Greg Not Designed By Roshan Frost Electronics 2025"
