File: Hardware/Vegan-Greg/VeganGreg.kicad_pcb (KiCad board)
At the start: 4 copper layers, 16 parts, among them U3 LM66200DRLR, U4 MAX77827AEFD+T, U5 SC4215ASTRT

Commit message: vegangreg pcb initial layout
Parts:
- added 12V: RED_LED, Resistor_SMD:R_0402_1005Metric, F.Cu at (173.9, 85.6)
- added 3V3: BLUE_LED, Resistor_SMD:R_0402_1005Metric, F.Cu at (171.4, 105.6)
- added BOOTJUMPER1: Conn_01x02_Male, Connector_PinHeader_2.54mm:PinHeader_1x02_P2.54mm_Vertical, F.Cu at (152.9, 124.1)
- added C1: 10uF, Capacitor_SMD:C_0402_1005Metric, F.Cu at (153.5, 117.6)
- added C10: 0.1uF, Capacitor_SMD:C_0402_1005Metric, F.Cu at (149.5, 109.1)
- added C11: 0.1uF, Capacitor_SMD:C_0402_1005Metric, F.Cu at (158.9, 115.6)
- added C12: 1uF, Capacitor_SMD:C_0402_1005Metric, F.Cu at (136.8, 93.7)
- added C13: 11pF, Capacitor_SMD:C_0402_1005Metric, F.Cu at (145.0, 110.1)
- added C14: 11pF, Capacitor_SMD:C_0402_1005Metric, F.Cu at (145.0, 114.1)
- added C15: 100nF, Capacitor_SMD:C_0402_1005Metric, F.Cu at (140.9, 105.1)
- added C16: 10uF, Capacitor_SMD:C_0402_1005Metric, F.Cu at (140.9, 104.1)
- added C17: 47nF, Capacitor_SMD:C_0402_1005Metric, F.Cu at (134.9, 112.6)
- added C18: 4.7uF, Capacitor_SMD:C_0402_1005Metric, F.Cu at (136.8, 92.7)
- added C19: 100uF, Capacitor_Tantalum_SMD:CP_EIA-7360-38_Kemet-E, F.Cu at (149.4, 93.6)
- added C2: 1uF, Capacitor_SMD:C_0402_1005Metric, F.Cu at (145.9, 124.1)
- added C28: 47uF, Capacitor_SMD:C_1206_3216Metric, F.Cu at (129.9, 103.6)
- added C29: 47uF, Capacitor_SMD:C_1206_3216Metric, F.Cu at (129.9, 101.1)
- added C3: 0.1uF, Capacitor_SMD:C_0402_1005Metric, F.Cu at (145.9, 123.1)
- added C30: 100nF, Capacitor_SMD:C_0402_1005Metric, F.Cu at (148.4, 97.6)
- added C31: 47uF, Capacitor_SMD:C_1206_3216Metric, F.Cu at (129.9, 98.6)
- added C32: 47uF, Capacitor_SMD:C_1206_3216Metric, F.Cu at (129.9, 96.1)
- added C33: 47uF, Capacitor_SMD:C_1206_3216Metric, F.Cu at (129.9, 93.6)
- added C34: 0.1uF, Capacitor_SMD:C_0402_1005Metric, F.Cu at (142.8, 97.7)
- added C35: 160pF, Capacitor_SMD:C_0603_1608Metric, F.Cu at (144.4, 89.6)
- added C4: 1uF, Capacitor_SMD:C_0402_1005Metric, F.Cu at (151.5, 117.6)
- added C42: 22µF, Capacitor_SMD:C_0603_1608Metric, F.Cu at (170.9, 88.1)
- added C43: 1µF, Capacitor_SMD:C_0402_1005Metric, F.Cu at (178.4, 87.1)
- added C44: 0.1µF, Capacitor_SMD:C_0402_1005Metric, F.Cu at (167.9, 85.6)
- added C45: 10uF, Capacitor_SMD:C_0402_1005Metric, F.Cu at (179.4, 89.1)
- added C46: 100nF, Capacitor_SMD:C_0402_1005Metric, F.Cu at (179.3, 88.1)
- added C47: 2.2µF, Capacitor_SMD:C_0402_1005Metric, F.Cu at (164.4, 87.6)
- added C48: 0.01µF, Capacitor_SMD:C_0402_1005Metric, F.Cu at (175.4, 90.6)
- added C49: 22µF, Capacitor_SMD:C_0603_1608Metric, F.Cu at (168.9, 91.1)
- added C5: 0.1uF, Capacitor_SMD:C_0402_1005Metric, F.Cu at (151.4, 116.6)
- added C50: 22µF, Capacitor_SMD:C_0603_1608Metric, F.Cu at (168.9, 92.6)
- added C51: 22µF, Capacitor_SMD:C_0603_1608Metric, F.Cu at (168.9, 94.1)
- added C52: 180pF, Capacitor_SMD:C_0402_1005Metric, F.Cu at (164.4, 88.6)
- added C53: 10µF, Capacitor_SMD:C_0402_1005Metric, F.Cu at (175.4, 89.6)
- added C54: 4.7nF, Capacitor_SMD:C_0402_1005Metric, F.Cu at (166.4, 90.6)
- added C55: 0.1uF, Capacitor_SMD:C_0402_1005Metric, F.Cu at (155.9, 89.1)
- added C6: 0.1uF, Capacitor_SMD:C_0402_1005Metric, F.Cu at (153.0, 116.1)
- added C7: 1uF, Capacitor_SMD:C_0402_1005Metric, F.Cu at (149.5, 114.6)
- added C8: 0.1uF, Capacitor_SMD:C_0402_1005Metric, F.Cu at (153.4, 121.6)
- added C9: 10nF, Capacitor_SMD:C_0402_1005Metric, F.Cu at (149.5, 113.6)
- added CRX: ORANGE_LED, Resistor_SMD:R_0402_1005Metric, F.Cu at (128.9, 110.6)
- added CTX: GREEN_LED, Resistor_SMD:R_0402_1005Metric, F.Cu at (135.9, 115.1)
- added D1: SM712_SOT23, Package_TO_SOT_SMD:SOT-23, F.Cu at (132.5, 109.6)
- added D2: SP0503BAHT, Package_TO_SOT_SMD:SOT-143, F.Cu at (172.9, 118.1)
- added D3: ~, Package_TO_SOT_SMD:SOT-353_SC-70-5, F.Cu at (152.4, 100.1)
- added D4: ~, Package_TO_SOT_SMD:SOT-353_SC-70-5, F.Cu at (152.3, 104.1)
- added D5: RCLAMP3346PQTNT, iclr:RCLAMP3346PQTNT, F.Cu at (157.8, 120.3)
- added ENJUMPER1: Conn_01x02_Male, Connector_PinHeader_2.54mm:PinHeader_1x02_P2.54mm_Vertical, F.Cu at (148.9, 124.1)
- added H1: MountingHole_Pad, MountingHole:MountingHole_3.2mm_M3_DIN965_Pad, F.Cu at (184.4, 79.6)
- added H2: MountingHole_Pad, MountingHole:MountingHole_3.2mm_M3_DIN965_Pad, F.Cu at (122.4, 79.3)
- added H3: MountingHole_Pad, MountingHole:MountingHole_3.2mm_M3_DIN965_Pad, F.Cu at (184.4, 124.6)
- added H4: MountingHole_Pad, MountingHole:MountingHole_3.2mm_M3_DIN965_Pad, F.Cu at (122.4, 124.3)
- added J1: RBUS, Connector_Molex:Molex_Mini-Fit_Jr_5566-06A_2x03_P4.20mm_Vertical, F.Cu at (141.1, 125.8)
- added J2: USB_C_Receptacle_USB2.0, Connector_USB:USB_C_Receptacle_Palconn_UTC16-G, F.Cu at (171.4, 123.7)
- added J3: ServoCH0, iclr:Molex_Nano-Fit_105313-xx03_1x03_P2.50mm_Horizontal, F.Cu at (152.9, 86.7)
- added J4: Conn_01x06_Socket, iclr:Molex_Mini-Fit_Jr_5569-06A2_2x03_P4.20mm_Horizontal, F.Cu at (181.7, 98.9)
- added J5: GPIO Breakout, Connector_PinSocket_2.54mm:PinSocket_2x04_P2.54mm_Vertical, F.Cu at (164.2, 126.6)
- added JP1: TermJP, Jumper:SolderJumper-2_P1.3mm_Open_RoundedPad1.0x1.5mm, F.Cu at (132.9, 106.6)
- added JP2: SolderJumper_3_Open, Jumper:SolderJumper-3_P1.3mm_Open_RoundedPad1.0x1.5mm_NumberLabels, F.Cu at (165.0, 94.1)
- added L1: 2.0nH, Inductor_SMD:L_0402_1005Metric, F.Cu at (151.5, 115.6)
- added L2: 20nH, Inductor_SMD:L_0402_1005Metric, F.Cu at (149.5, 112.6)
- added L4: 3.3uH, iclr:IND_SPM10065VT-3R3M-D, F.Cu at (136.4, 85.1)
- added L5: 1.8µH, Inductor_SMD:L_0805_2012Metric, F.Cu at (170.9, 86.1)
- added LED1: WHITE_LED, Resistor_SMD:R_0402_1005Metric, F.Cu at (168.3, 119.1)
- added Q1: SSM3K15AMFV,L3F, iclr:SOT-723, F.Cu at (146.4, 105.6)
- added R1: 10K, Resistor_SMD:R_0402_1005Metric, F.Cu at (148.4, 121.6)
- added R10: 60, Resistor_SMD:R_0603_1608Metric, F.Cu at (140.4, 112.6)
- added R11: 5.1k, Resistor_SMD:R_0402_1005Metric, F.Cu at (170.3, 119.1)
- added R12: 5.1k, Resistor_SMD:R_0402_1005Metric, F.Cu at (178.3, 121.1)
- added R13: 5.1k, Resistor_SMD:R_0402_1005Metric, F.Cu at (169.3, 119.1)
- added R18: 1k, Resistor_SMD:R_0402_1005Metric, F.Cu at (128.9, 111.6)
- added R19: 165R, Resistor_SMD:R_0402_1005Metric, F.Cu at (155.4, 105.1)
- added R2: 470, Resistor_SMD:R_0402_1005Metric, F.Cu at (130.9, 115.1)
- added R20: 10k, Resistor_SMD:R_0402_1005Metric, F.Cu at (135.3, 93.2)
- added R21: 113k, Resistor_SMD:R_0402_1005Metric, F.Cu at (136.4, 98.1)
- added R22: 10k, Resistor_SMD:R_0402_1005Metric, F.Cu at (136.4, 97.1)
- added R23: 2.2, Resistor_SMD:R_0402_1005Metric, F.Cu at (144.8, 97.7)
- added R24: 1k, Resistor_SMD:R_0402_1005Metric, F.Cu at (148.4, 105.6)
- added R25: 442k, Resistor_SMD:R_0402_1005Metric, F.Cu at (134.9, 97.6)
- added R26: 200k, Resistor_SMD:R_0402_1005Metric, F.Cu at (139.4, 97.6)
- added R27: 100k, Resistor_SMD:R_0402_1005Metric, F.Cu at (141.3, 98.2)
- added R28: 10k, Resistor_SMD:R_0402_1005Metric, F.Cu at (145.9, 102.1)
- added R29: 5.1R, Resistor_SMD:R_0603_1608Metric, F.Cu at (144.4, 88.1)
- added R3: 10K, Resistor_SMD:R_0402_1005Metric, F.Cu at (151.9, 121.1)
- added R30: 301k, Resistor_SMD:R_0402_1005Metric, F.Cu at (165.4, 84.1)
- added R31: 127k, Resistor_SMD:R_0402_1005Metric, F.Cu at (170.4, 89.6)
- added R32: 17.4k, Resistor_SMD:R_0402_1005Metric, F.Cu at (164.9, 90.1)
- added R33: 100k, Resistor_SMD:R_0402_1005Metric, F.Cu at (168.2, 96.6)
- added R34: 51k, Resistor_SMD:R_0402_1005Metric, F.Cu at (166.7, 96.6)
- added R35: 18k, Resistor_SMD:R_0402_1005Metric, F.Cu at (165.2, 96.6)
- added R36: 18k, Resistor_SMD:R_0402_1005Metric, F.Cu at (133.9, 91.1)
- added R37: 1.5k, Resistor_SMD:R_0402_1005Metric, F.Cu at (155.9, 90.6)
- added R38: 470, Resistor_SMD:R_0402_1005Metric, F.Cu at (155.9, 92.1)
- added R39: 1k, Resistor_SMD:R_0402_1005Metric, F.Cu at (155.9, 93.6)
- added R4: 470, Resistor_SMD:R_0402_1005Metric, F.Cu at (171.4, 104.6)
- added R5: 1k, Resistor_SMD:R_0402_1005Metric, F.Cu at (135.9, 114.1)
- added R6: 499R, Resistor_SMD:R_0402_1005Metric, F.Cu at (149.5, 110.1)
- added R7: 3k, Resistor_SMD:R_0402_1005Metric, F.Cu at (173.9, 86.6)
- added R8: 0, Resistor_SMD:R_0603_1608Metric, F.Cu at (140.4, 115.6)
- added R9: 60, Resistor_SMD:R_0603_1608Metric, F.Cu at (140.4, 114.1)
- added SERVOLED1: AMBER_LED, LED_SMD:LED_0402_1005Metric, F.Cu at (155.9, 95.1)
- added TP1: TestPoint, TestPoint:TestPoint_Pad_D1.0mm, F.Cu at (174.4, 115.1)
- added TP10: TestPoint, TestPoint:TestPoint_Pad_D1.0mm, F.Cu at (147.4, 117.1)
- added TP2: TestPoint, TestPoint:TestPoint_Pad_D1.0mm, F.Cu at (171.9, 115.1)
- added TP4: TestPoint, TestPoint:TestPoint_Pad_D1.5mm, F.Cu at (163.9, 115.6)
- added TP5: TestPoint, TestPoint:TestPoint_Pad_D1.5mm, F.Cu at (181.4, 113.1)
- added TP6: TestPoint, TestPoint:TestPoint_Pad_D1.5mm, F.Cu at (177.9, 113.6)
- added TP8: TestPoint, TestPoint:TestPoint_Pad_D1.5mm, F.Cu at (160.9, 97.6)
- added TP9: TestPoint, TestPoint:TestPoint_Pad_D1.0mm, F.Cu at (147.4, 108.6)
- added TX: GREEN_LED, Resistor_SMD:R_0402_1005Metric, F.Cu at (130.9, 114.1)
- added U1: ESP32-S3, iclr:QFN40P700X700X90-57N, F.Cu at (155.0, 110.6)
- added U2: SN65HVD230, Package_SO:SOIC-8_3.9x4.9mm_P1.27mm, F.Cu at (138.4, 108.6)
- added U6: SIC438AED-T1, iclr:SiC437BEDT1GE3, F.Cu at (141.3, 93.7)
- added U7: LT1762, Package_SO:MSOP-8_3x3mm_P0.65mm, F.Cu at (176.9, 93.1)
- added U8: TPS61089, Package_DFN_QFN:Texas_VQFN-RNR0011A-11, F.Cu at (167.2, 87.8)
- added Y1: R940000171, Crystal:Crystal_SMD_2016-4Pin_2.0x1.6mm, F.Cu at (145.0, 112.1)
- moved C24 26.8 mm to (159.7, 100.9), turned to 90 degrees
- moved C20 26.8 mm to (161.9, 111.2), turned to 180 degrees
- moved C25 26.8 mm to (159.7, 103.0), turned to -90 degrees
- moved U3 26.4 mm to (163.3, 113.0), turned to 0 degrees
- moved R15 26.3 mm to (161.0, 108.2), turned to -90 degrees
- moved C22 26.2 mm to (161.9, 110.3), turned to 180 degrees
- moved R14 23.2 mm to (165.5, 112.2), turned to 180 degrees
- moved U4 23.2 mm to (163.3, 108.1), turned to 0 degrees
- moved C21 22.9 mm to (164.7, 110.6), turned to 0 degrees
- moved U5 20.9 mm to (163.9, 102.0), turned to 0 degrees
- moved C23 20.5 mm to (164.5, 105.5), turned to 0 degrees
- moved L3 18.3 mm to (167.1, 108.1), turned to 90 degrees
- moved C26 15.8 mm to (168.1, 104.7), turned to 90 degrees
- moved R17 15.7 mm to (168.1, 101.0), turned to 90 degrees
- moved R16 15.5 mm to (168.1, 102.9), turned to 90 degrees
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
Commit message: Full PCB design
Parts:
- removed D3: ~, Package_TO_SOT_SMD:SOT-353_SC-70-5
- added C56: 10nF, Capacitor_SMD:C_0402_1005Metric, F.Cu at (134.9, 103.1)
- added C58: 220nF, Capacitor_SMD:C_0402_1005Metric, F.Cu at (141.5, 102.1)
- added C59: 1nF, Capacitor_SMD:C_0402_1005Metric, F.Cu at (140.5, 101.1)
- added C60: 1nF, Capacitor_SMD:C_0402_1005Metric, F.Cu at (139.5, 102.1)
- added C61: 0.1uF, Capacitor_SMD:C_0402_1005Metric, F.Cu at (163.4, 119.1)
- added J7: ST1W008S4TR2000, iclr:JAE_ST1W008S4TR2000, F.Cu at (177.4, 122.6)
- added JP13: SolderJumper_2_Open, iclr:SmallerSolderJP, F.Cu at (163.9, 117.1)
- added JP4: SolderJumper_3_Open, Jumper:SolderJumper-3_P1.3mm_Open_RoundedPad1.0x1.5mm_NumberLabels, F.Cu at (130.4, 105.9)
- added JP5: SolderJumper_3_Open, Jumper:SolderJumper-3_P1.3mm_Open_RoundedPad1.0x1.5mm_NumberLabels, F.Cu at (132.9, 105.8)
- added JP6: SolderJumper_2_Open, iclr:SmallerSolderJP, F.Cu at (131.9, 101.1)
- added JP7: SolderJumper_2_Open, iclr:SmallerSolderJP, F.Cu at (129.9, 101.1)
- added Q2: PMOS, Package_TO_SOT_SMD:SOT-23, F.Cu at (165.9, 119.6)
- added R46: 75k, Resistor_SMD:R_0402_1005Metric, F.Cu at (131.4, 109.1)
- added R47: 14k, Resistor_SMD:R_0402_1005Metric, F.Cu at (134.9, 107.1)
- added R48: 10k, Resistor_SMD:R_0402_1005Metric, F.Cu at (134.9, 105.1)
- added R49: 1k, Resistor_SMD:R_0402_1005Metric, F.Cu at (134.9, 101.1)
- added R50: 49.9, Resistor_SMD:R_0402_1005Metric, F.Cu at (130.9, 99.4)
- added R51: 1k, Resistor_SMD:R_0402_1005Metric, F.Cu at (133.9, 102.1)
- added R52: 54.9, Resistor_SMD:R_0402_1005Metric, F.Cu at (151.4, 105.6)
- added R59: 1k, Resistor_SMD:R_0402_1005Metric, F.Cu at (166.9, 121.9)
- added R60: 10k, Resistor_SMD:R_0402_1005Metric, F.Cu at (164.9, 121.9)
- added U9: ADS131M02IRUKR, footprints:WQFN20_ADS131_TEX, F.Cu at (140.7, 105.0)
- J1: footprint Connector_Molex:Molex_Mini-Fit_Jr_5566-06A_2x03_P4.20mm_Vertical -> iclr:Molex_Mini-Fit_Jr_5569-06A2_2x03_P4.20mm_Horizontal
- J4: value Conn_01x06_Socket -> 1053131104; footprint iclr:Molex_Mini-Fit_Jr_5569-06A2_2x03_P4.20mm_Horizontal -> Connector_Molex:Molex_Nano-Fit_105313-xx04_1x04_P2.50mm_Horizontal
- moved C48 56.5 mm to (122.4, 110.1)
- moved C53 56.5 mm to (122.4, 109.1)
- moved L5 56.5 mm to (120.9, 112.3), turned to -90 degrees
- moved C44 56.0 mm to (120.4, 115.3), turned to 90 degrees
- moved R30 55.9 mm to (120.4, 117.3), turned to -90 degrees
- moved J4 55.0 mm to (127.1, 105.8), turned to 180 degrees
- moved C42 53.8 mm to (122.9, 112.4), turned to -90 degrees
- moved C45 53.3 mm to (131.9, 113.6)
- moved C46 53.3 mm to (131.9, 112.6)
- moved U7 52.8 mm to (126.9, 110.1)
- moved C43 52.8 mm to (131.4, 111.1)
- moved C47 52.7 mm to (121.9, 118.8), turned to -90 degrees
- moved U8 52.7 mm to (122.7, 116.0), turned to 90 degrees
- moved R31 51.7 mm to (124.9, 114.1), turned to 90 degrees
- moved C52 50.9 mm to (123.4, 118.8), turned to -90 degrees
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- renumbered 12V to 12VLED1, 3V3 to 3V3LED1, CRX to CRXLED1, CTX to CTXLED1, TX to TXLED1, LED1 to USBLED1
Connections:
- C19 pad 1: +16.8V -> DeployV
- C30 pad 1: +16.8V -> DeployV
- C43 pad 1: Net-(U7-IN) -> 5_or_12
- C45 pad 1: /gregPart/LDO5.5V_IN -> 5_or_12
- C46 pad 1: /gregPart/LDO5.5V_IN -> 5_or_12
- C48 pad 1: Net-(U7-ADJ) -> LDO_out
- C49 pad 1: /gregPart/VOut - 5 or 12V -> 5_or_12
- C50 pad 1: /gregPart/VOut - 5 or 12V -> 5_or_12
- C51 pad 1: /gregPart/VOut - 5 or 12V -> 5_or_12
- C53 pad 1: Net-(U7-ADJ) -> LDO_out
- J1 pad 4: +25.2V -> DeployV
- J4 pad 1: GND -> LDO_out
- J4 pad 2: GND -> Net-(JP4-C)
- J4 pad 3: RBUS_uC_V -> Net-(JP7-B)
- J4 pad 4: +12V -> GND
- R28 pad 2: +16.8V -> DeployV
- R34 pad 1: /gregPart/VOut - 5 or 12V -> 5_or_12
- R7 pad 1: 25.2V -> DeployV
- U1 pad 16: unconnected-(U1-GPIO11/ADC2_CH0-Pad16) -> /SD_DET
- U1 pad 17: unconnected-(U1-GPIO12/ADC2_CH1-Pad17) -> /SD_EN
- U1 pad 18: unconnected-(U1-GPIO13/ADC2_CH2-Pad18) -> /SD_CS
- U1 pad 19: unconnected-(U1-GPIO14/ADC2_CH3-Pad19) -> /VSPI_MOSI
- U1 pad 23: unconnected-(U1-GPIO17/ADC2_CH6/DAC_2-Pad23) -> /VSPI_SCLK
- U1 pad 24: unconnected-(U1-GPIO18/ADC2_CH7/DAC_1-Pad24) -> /VSPI_MISO
- U1 pad 36: unconnected-(U1-SPICLK_N/GPIO48-Pad36) -> /CAN_RX
- U1 pad 37: /BuckPGOOD -> /CAN_TX
- U1 pad 38: /CAN_TX -> /BUCK_EN
- U1 pad 39: /CAN_RX -> /BuckPGOOD
- U1 pad 42: unconnected-(U1-GPIO37-Pad42) -> Net-(U1-GPIO37)
- U1 pad 43: /BUCK_EN -> /ADS_MOSI
- U1 pad 44: unconnected-(U1-MTCK/JTAG/GPIO39-Pad44) -> /ADS_MISO
- U1 pad 45: unconnected-(U1-MTDO/JTAG/GPIO40-Pad45) -> /ADS_SCLK
- U1 pad 47: unconnected-(U1-MTDI/JTAG/GPIO41-Pad47) -> /ADS_DRDY
- U1 pad 48: unconnected-(U1-MTMS/JTAG/GPIO42-Pad48) -> /ADS_CS
- U6 pad 1: +16.8V -> DeployV
- U6 pad 2: +16.8V -> DeployV
- U6 pad 22: +16.8V -> DeployV
- U6 pad 26: +16.8V -> DeployV
- U7 pad 1: Net-(U7-ADJ) -> LDO_out
- U7 pad 2: Net-(U7-ADJ) -> LDO_out
- U7 pad 5: Net-(U7-IN) -> 5_or_12
- U7 pad 8: Net-(U7-IN) -> 5_or_12
- U8 pad 6: /gregPart/VOut - 5 or 12V -> 5_or_12
Routing:
- net GND: track 7.31 -> 202.4 mm, vias 8 -> 64
- net +3V3: track 1.61 -> 110.5 mm, vias 1 -> 11
- net RBUS_uC_V: track 0.00 -> 65.1 mm, vias 0 -> 2
- net VBUS: track 5.51 -> 63.7 mm, vias 2 -> 3
- net +6V: track 0.00 -> 54.8 mm, vias 0 -> 4
- net /SD_DET: track 0.00 -> 46.1 mm
- net /Data+: track 0.00 -> 33.9 mm
- net /Data-: track 0.00 -> 33.5 mm
- net DeployV: track 0.00 -> 31.8 mm
- net +3.3V: track 0.00 -> 30.5 mm, vias 0 -> 3
- net Net-(J3-Pin_3): track 0.00 -> 27.2 mm
- net /VSPI_MOSI: track 0.00 -> 23.3 mm
- net /SD_CS: track 0.00 -> 23.0 mm
- net /VSPI_MISO: track 0.00 -> 23.0 mm
- net /VSPI_SCLK: track 0.00 -> 22.7 mm
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- added copper zone on In2.Cu, net +3.3V
- added copper zone on B.Cu, net GND
- added copper zone on In1.Cu, net GND
Other:
- board outline added: 78 x 54 mm
